File: electronics/ClimateController/ClimateController.kicad_sch (KiCad schematic)
At the start: 22 parts, among them J2 UCB-C Breakout, J3 Conn_01x03, K1 FINDER-30.22, Q3 BC547, U1 ESP-12F, U2 AMS1117-3.3, U5 DHT11

Commit message: Rename KiCad files
Parts:
- C1: value 10uF -> 100nF; footprint (none) -> Capacitor_SMD:C_1210_3225Metric_Pad1.33x2.70mm_HandSolder
- C2, C3: renamed from C1; footprint (none) -> Capacitor_SMD:C_1210_3225Metric_Pad1.33x2.70mm_HandSolder
- D1: footprint Diode_THT:D_DO-41_SOD81_P10.16mm_Horizontal -> Diode_SMD:D_SMA_Handsoldering
- J1: renamed from J2; value UCB-C Breakout -> E-Paper; footprint (none) -> Connector_JST:JST_PH_B8B-PH-K_1x08_P2.00mm_Vertical
- J2: value UCB-C Breakout -> IR Emitter; footprint (none) -> Connector_JST:JST_PH_B3B-PH-K_1x03_P2.00mm_Vertical
- J3: renamed from J2; footprint (none) -> AA_Footprints:USB-C Breakout
- J4: renamed from J2; value UCB-C Breakout -> Serial Terminals; footprint (none) -> Connector_JST:JST_PH_B6B-PH-K_1x06_P2.00mm_Vertical
- J5: renamed from J3; value Conn_01x03 -> Heater Phase; footprint (none) -> TerminalBlock:TerminalBlock_bornier-3_P5.08mm
- Q1: renamed from Q3; footprint Package_TO_SOT_THT:TO-92_Inline -> Package_TO_SOT_SMD:SOT-23
- R1: footprint (none) -> Resistor_SMD:R_1206_3216Metric_Pad1.30x1.75mm_HandSolder
- R2, R3, R4, R5, R7: renamed from R1; footprint (none) -> Resistor_SMD:R_1206_3216Metric_Pad1.30x1.75mm_HandSolder
- R6: renamed from R1; value 10K -> 1K; footprint (none) -> Resistor_SMD:R_1206_3216Metric_Pad1.30x1.75mm_HandSolder
- U2: renamed from U1; footprint (none) -> AA_Footprints:ESP-12E_SMD
- renumbered U5 to U1, U2 to U3

Commit message: Improve file naming & Design V2 Dimmer iteration & Lay components in PCB
Other:
- title: Temperature Controller -> Climate Controller
Changed lines of the file:
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@@
   (paper "A4")
   (title_block
-    (title "Temperature Controller")
+    (title "Climate Controller")
     (date "2022-09-05")
     (rev "v2.0.0")
     (company "Pablo Ortiz")
+    (comment 1 "ortizma.com")
+    (comment 2 "Controls the Temperature and monitors the air quality in a room")
+    (comment 3 "Supports CO2 Readings via Serial")
+    (comment 4 "Supports controlling Climate units via IR and a relay")
   )
   (junction (at 242.57 46.99) (diameter 0) (color 0 0 0 0)
@@
     (pin "2")
     (instances
-      (project "ac-control"
+      (project "ClimateController"
         (path "/3d8b4ce2-7f39-402d-99e1-eee55263149f"
           (reference "D2") (unit 1)
@@
     (pin "1")
     (instances
-      (project "ac-control"
+      (project "ClimateController"
         (path "/3d8b4ce2-7f39-402d-99e1-eee55263149f"
           (reference "#PWR03") (unit 1)
@@
     (pin "1")
     (instances
-      (project "ac-control"
+      (project "ClimateController"
         (path "/3d8b4ce2-7f39-402d-99e1-eee55263149f"
           (reference "#PWR0107") (unit 1)
@@
     (pin "9")
     (instances
-      (project "ac-control"
+      (project "ClimateController"
         (path "/3d8b4ce2-7f39-402d-99e1-eee55263149f"
           (reference "U2") (unit 1)
@@
     (pin "2")
     (instances
-      (project "ac-control"
+      (project "ClimateController"
         (path "/3d8b4ce2-7f39-402d-99e1-eee55263149f"
           (reference "R7") (unit 1)
@@
     (pin "6")
     (instances
-      (project "ac-control"
+      (project "ClimateController"
         (path "/3d8b4ce2-7f39-402d-99e1-eee55263149f"
           (reference "J4") (unit 1)
@@
     (pin "1")
     (instances
-      (project "ac-control"
+      (project "ClimateController"
         (path "/3d8b4ce2-7f39-402d-99e1-eee55263149f"
           (reference "#PWR015") (unit 1)
@@
     (pin "1")
     (instances
-      (project "ac-control"
+      (project "ClimateController"
         (path "/3d8b4ce2-7f39-402d-99e1-eee55263149f"
           (reference "#PWR0106") (unit 1)
@@
     (pin "1")
     (instances
-      (project "ac-control"
+      (project "ClimateController"
         (path "/3d8b4ce2-7f39-402d-99e1-eee55263149f"
           (reference "#PWR0102") (unit 1)
@@
     (pin "6")
     (instances
-      (project "ac-control"
+      (project "ClimateController"
         (path "/3d8b4ce2-7f39-402d-99e1-eee55263149f"
           (reference "J3") (unit 1)
@@
     (pin "1")
     (instances
-      (project "ac-control"
+      (project "ClimateController"
         (path "/3d8b4ce2-7f39-402d-99e1-eee55263149f"
           (reference "#PWR011") (unit 1)
@@
     (pin "3")
     (instances
-      (project "ac-control"
+      (project "ClimateController"
         (path "/3d8b4ce2-7f39-402d-99e1-eee55263149f"
           (reference "J2") (unit 1)
@@
     (pin "2")
     (instances
-      (project "ac-control"
+      (project "ClimateController"
         (path "/3d8b4ce2-7f39-402d-99e1-eee55263149f"
           (reference "C2") (unit 1)
@@
     (pin "1")
     (instances
-      (project "ac-control"
+      (project "ClimateController"
         (path "/3d8b4ce2-7f39-402d-99e1-eee55263149f"
           (reference "#PWR02") (unit 1)
@@
     (pin "3")
     (instances
-      (project "ac-control"
+      (project "ClimateController"
         (path "/3d8b4ce2-7f39-402d-99e1-eee55263149f"
           (reference "J5") (unit 1)
@@
     (pin "1")
     (instances
-      (project "ac-control"
+      (project "ClimateController"
         (path "/3d8b4ce2-7f39-402d-99e1-eee55263149f"
           (reference "#PWR017") (unit 1)
@@
     (pin "1")
     (instances
-      (project "ac-control"
+      (project "ClimateController"
         (path "/3d8b4ce2-7f39-402d-99e1-eee55263149f"
           (reference "#PWR018") (unit 1)
@@
     (pin "1")
     (instances
-      (project "ac-control"
+      (project "ClimateController"
         (path "/3d8b4ce2-7f39-402d-99e1-eee55263149f"
           (reference "#PWR0105") (unit 1)
@@
     (pin "1")
     (instances
-      (project "ac-control"
+      (project "ClimateController"
         (path "/3d8b4ce2-7f39-402d-99e1-eee55263149f"
           (reference "#PWR06") (unit 1)
@@
     (pin "2")
     (instances
-      (project "ac-control"
+      (project "ClimateController"
         (path "/3d8b4ce2-7f39-402d-99e1-eee55263149f"
           (reference "R6") (unit 1)
@@
     (pin "2")
     (instances
-      (project "ac-control"
+      (project "ClimateController"
         (path "/3d8b4ce2-7f39-402d-99e1-eee55263149f"
           (reference "D1") (unit 1)
@@
     (pin "2")
     (instances
-      (project "ac-control"
+      (project "ClimateController"
         (path "/3d8b4ce2-7f39-402d-99e1-eee55263149f"
           (reference "R1") (unit 1)
@@
     (pin "2")
     (instances
-      (project "ac-control"
+      (project "ClimateController"
         (path "/3d8b4ce2-7f39-402d-99e1-eee55263149f"
           (reference "R5") (unit 1)
@@
     (pin "1")
     (instances
-      (project "ac-control"
+      (project "ClimateController"
         (path "/3d8b4ce2-7f39-402d-99e1-eee55263149f"
           (reference "#PWR014") (unit 1)
@@
     (pin "1")
     (instances
-      (project "ac-control"
+      (project "ClimateController"
         (path "/3d8b4ce2-7f39-402d-99e1-eee55263149f"
           (reference "#PWR016") (unit 1)
@@
     (pin "8")
     (instances
-      (project "ac-control"
+      (project "ClimateController"
         (path "/3d8b4ce2-7f39-402d-99e1-eee55263149f"
           (reference "J1") (unit 1)
@@
     (pin "2")
     (instances
-      (project "ac-control"
+      (project "ClimateController"
         (path "/3d8b4ce2-7f39-402d-99e1-eee55263149f"
           (reference "R2") (unit 1)
@@
     (pin "1")
     (instances
-      (project "ac-control"
+      (project "ClimateController"
         (path "/3d8b4ce2-7f39-402d-99e1-eee55263149f"
           (reference "#PWR0108") (unit 1)
@@
     (pin "2")
     (instances
-      (project "ac-control"
+      (project "ClimateController"
         (path "/3d8b4ce2-7f39-402d-99e1-eee55263149f"
           (reference "R4") (unit 1)
@@
     (pin "3")
     (instances
-      (project "ac-control"
+      (project "ClimateController"
         (path "/3d8b4ce2-7f39-402d-99e1-eee55263149f"
           (reference "U3") (unit 1)
@@
     (pin "2")
     (instances
-      (project "ac-control"
+      (project "ClimateController"
         (path "/3d8b4ce2-7f39-402d-99e1-eee55263149f"
           (reference "R3") (unit 1)
@@
     (pin "2")
     (instances
-      (project "ac-control"
+      (project "ClimateController"
         (path "/3d8b4ce2-7f39-402d-99e1-eee55263149f"
           (reference "C3") (unit 1)
@@
     (pin "1")
     (instances
-      (project "ac-control"
+      (project "ClimateController"
         (path "/3d8b4ce2-7f39-402d-99e1-eee55263149f"
           (reference "#PWR01") (unit 1)
@@
     (pin "4")
     (instances
-      (project "ac-control"
+      (project "ClimateController"
         (path "/3d8b4ce2-7f39-402d-99e1-eee55263149f"
           (reference "U1") (unit 1)
@@
     (pin "2")
     (instances
-      (project "ac-control"
+      (project "ClimateController"
         (path "/3d8b4ce2-7f39-402d-99e1-eee55263149f"
           (reference "C1") (unit 1)
@@
     (pin "1")
     (instances
-      (project "ac-control"
+      (project "ClimateController"
         (path "/3d8b4ce2-7f39-402d-99e1-eee55263149f"
           (reference "#PWR021") (unit 1)
@@
     (pin "3")
     (instances
-      (project "ac-control"
+      (project "ClimateController"
         (path "/3d8b4ce2-7f39-402d-99e1-eee55263149f"
           (reference "Q1") (unit 1)
@@
     (pin "1")
     (instances
-      (project "ac-control"
+      (project "ClimateController"
         (path "/3d8b4ce2-7f39-402d-99e1-eee55263149f"
           (reference "#PWR0103") (unit 1)
@@
     (pin "1")
     (instances
-      (project "ac-control"
+      (project "ClimateController"
         (path "/3d8b4ce2-7f39-402d-99e1-eee55263149f"
           (reference "#PWR08") (unit 1)
@@
     (pin "1")
     (instances
-      (project "ac-control"
+      (project "ClimateController"
         (path "/3d8b4ce2-7f39-402d-99e1-eee55263149f"
           (reference "#PWR0104") (unit 1)
@@
     (pin "1")
     (instances
-      (project "ac-control"
+      (project "ClimateController"
         (path "/3d8b4ce2-7f39-402d-99e1-eee55263149f"
           (reference "#PWR0101") (unit 1)
@@
     (pin "1")
     (instances
-      (project "ac-control"
+      (project "ClimateController"
         (path "/3d8b4ce2-7f39-402d-99e1-eee55263149f"
           (reference "#PWR04") (unit 1)
@@
     (pin "1")
     (instances
-      (project "ac-control"
+      (project "ClimateController"
         (path "/3d8b4ce2-7f39-402d-99e1-eee55263149f"
           (reference "#PWR010") (unit 1)
@@
     (pin "A2")
     (instances
-      (project "ac-control"
+      (project "ClimateController"
         (path "/3d8b4ce2-7f39-402d-99e1-eee55263149f"
           (reference "K1") (unit 1)
@@
     (pin "1")
     (instances
-      (project "ac-control"
+      (project "ClimateController"
         (path "/3d8b4ce2-7f39-402d-99e1-eee55263149f"
           (reference "#PWR05") (unit 1)
