File: electronics/LightDimmer/LightDimmer.kicad_sch (KiCad schematic)
At the start: 12 parts, among them J2 AC Terminals, J4 Serial Terminals, U2 5V07, U2 ESP-12F, U3 AC Dimmer 4A

Commit message: Rename KiCad files
Parts:
- added D1: 1N4007, Diode_THT:D_DO-41_SOD81_P10.16mm_Horizontal, symbol Diode:1N4007
- added K1: SANYOU_SRD_Form_C, Relay_THT:Relay_SPDT_SANYOU_SRD_Series_Form_C, symbol Relay:SANYOU_SRD_Form_C
- added Q1: BC547, Package_TO_SOT_THT:TO-92_Inline, symbol Transistor_BJT:BC547
- added R6: 1k, symbol Device:R_Small
Connections:
- net +3.3V: now also D1.1 (K), K1.5
- net GND: now also Q1.3 (E)
- net GPIO5: now also R6.1
- net LAMP: now also K1.1; no longer U3.7 (OUT)
- net AC renamed LINE
- new net: D1.2 (A), K1.2, Q1.1 (C)
- new net: Q1.2 (B), R6.2
- new net DIMMER_OUT: K1.3, U3.7 (OUT)
Other:
- company: (none) -> Pablo Ortiz López
- title: (none) -> Wi-Fi + RF AC Dimmer
- moved on the sheet: C1, R1, R2, R3, R4, R5, U2, U3

Commit message: Add RF receiver in Dimmer
Parts:
- added J3: 433MHz_ASK_Superheterodyne_Receiver, symbol 00_Symbols:433MHz_ASK_Superheterodyne_Receiver
Connections:
- net +3.3V: now also J3.4 (VCC)
- net GND: now also J3.1 (GND)
- net GPIO14: now also J3.2 (DATA), J3.3 (DATA)

Commit message: Improve file naming & Design V2 Dimmer iteration & Lay components in PCB
Parts:
- D1: footprint Diode_THT:D_DO-41_SOD81_P10.16mm_Horizontal -> Diode_SMD:D_SMA_Handsoldering
- J1: renamed from J3; footprint (none) -> AA_Footprints:RF Receiver
- J3: renamed from J2; footprint TerminalBlock:TerminalBlock_bornier-4_P5.08mm -> AA_Footprints:Terminal_KF128-4P
- Q1: footprint Package_TO_SOT_THT:TO-92_Inline -> AA_Footprints:SOT-23-3-BC
- R6: footprint (none) -> Resistor_SMD:R_1206_3216Metric_Pad1.30x1.75mm_HandSolder
- U1: renamed from U2; value 5V07 -> 5V07 Transformer; symbol 5V07:5V07 -> 00_Symbols:5V07
- U3: value AC Dimmer 4A -> AC_Dimmer_4A; symbol AC Dimmer 4A:AC_Dimmer_4A -> 00_Symbols:AC_Dimmer_4A

Commit message: Improved the designs of LightController & LightDimmer PCBs
Parts:
- U2: footprint AA_Footprints:ESP-12E_SMD -> AA_Footprints:ESP-12E_SMD_Simple
Changed lines of the file:
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@@
       (effects (font (size 1.27 1.27)))
     )
-    (property "Footprint" "AA_Footprints:ESP-12E_SMD" (at 104.14 41.91 0)
+    (property "Footprint" "AA_Footprints:ESP-12E_SMD_Simple" (at 104.14 41.91 0)
       (effects (font (size 1.27 1.27)) hide)
     )
